File: ESP8266Shield/ESP8266Shield.brd (EAGLE design)
At the start: 49.2 x 48.3 mm, 19 parts, among them IC1 MEGA8-P, Q1 2N5088, Q2 2N5088

Commit message: v0.06
Added Shield schematic, and gerber files.
It has not yet been verified.
Parts:
- added JP5, JP6: (no value), SparkFun:1X08
- added JP8, JP9: USB to Serial, SparkFun:1X06
- moved ESP8266 2.84 mm to (38.1, 33.0)
- moved Q2 1.80 mm to (47.8, 38.1)
- moved U$2 1.27 mm to (59.7, 36.1)
Connections:
- new net N$5: JP2.7, JP6.7
- new net N$6: JP2.8, JP6.8
- new net N$7: JP4.6, JP8.6
- net 3.3V: now also JP8.2
- net D0: now also JP5.1
- net D1: now also JP5.2
- net D10: now also JP6.3
- net D11: now also JP6.4
- net D12: now also JP6.5
- net D13: now also JP6.6
- net D14: now also JP9.1
- net D15: now also JP9.2
- net D16: now also JP9.3
- net D17: now also JP9.4
- net D18: now also JP9.5
- net D19: now also JP9.6
- net D2: now also JP5.3
- net D3: now also JP5.4
- net D4: now also JP5.5
- net D5: now also JP5.6
- net D6: now also JP5.7
- net D7: now also JP5.8
- net D8: now also JP6.1
- net D9: now also JP6.2
- net GND: now also JP8.4, JP8.5
- net RESET: now also JP8.1
- net VCC: now also JP8.3
Routing:
- net D5: track 31.0 -> 71.9 mm, vias 2 -> 6
- net GND: track 113.7 -> 147.7 mm, vias 0 -> 2
- net D8: track 32.7 -> 50.2 mm, vias 1 -> 0
- net VCC: track 111.9 -> 128.5 mm
- net 3.3V: track 73.9 -> 61.8 mm, vias 0 -> 2
- net RESET: track 63.1 -> 71.1 mm, vias 2 -> 0
- net N$3: track 32.2 -> 25.0 mm, vias 1 -> 0
- net D12: track 23.9 -> 31.1 mm, vias 0 -> 1
- net D13: track 37.5 -> 30.4 mm
- net D7: track 31.7 -> 37.6 mm, vias 1 -> 0
- net ESPRX: track 28.2 -> 33.9 mm
- net D16: track 27.8 -> 33.4 mm, vias 0 -> 1
- net D9: track 34.0 -> 39.4 mm, vias 2 -> 0
- net N$5: track 0.00 -> 2.89 mm
- net N$6: track 0.00 -> 2.86 mm
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